File: ETeam.kicad_pcb (KiCad board)
At the start: 2 copper layers, 445.3 x 72 mm, 276 parts, among them IC1 LT3990, IC2 LTC6804-2, IC3 LT3990, IC4 LTC6804-2, IC5 LT3990, IC6 LTC6804-2, J1 C1-, J12 C28+, J13 C27+, J14 C26+, J15 C25+, J16 C23+, J17 C22+, J18 C21+, J19 C20+, J2 C12+, J20 C19+, J21 C18+, J22 C17+, J23 C16+, J24 C15+, J25 C14+, J26 C13+, J27 C11+, J28 C10+, J29 C9+, J3 C24+, J30 C8+, J31 C7+, J32 C6+, J33 C5+, J34 C4+, J35 C3+, J36 C2+, J37 C1+, P1 BUS_OUT, P10 T29-32, P2 BUS_IN, P3 T1-4, P4 T5-8, P5 T9-12, P6 T13-16, P7 T17-20, P8 T21-24, P9 T25-28, Q10 BSS308, Q11 BSS308, Q12 BSS308, Q13 BSS308, Q14 BSS308, Q15 BSS308, Q16 BSS308, Q17 BSS308, Q18 BSS308, Q19 BSS308, Q20 BSS308, Q21 BSS308, Q22 BSS308, Q23 BSS308, Q24 BSS308, Q25 Q_NMOS_GSD, Q26 BSS308, Q27 BSS308, Q28 BSS308, Q29 BSS308, Q30 BSS308, Q31 BSS308, Q32 BSS308, Q33 BSS308, Q34 BSS308, Q35 BSS308, Q36 BSS308, Q37 BSS308, Q38 Q_NMOS_GSD, Q9 BSS308, SW1 Coded_Switch, SW2 Coded_Switch, SW3 Coded_Switch, T1 ACT45B-220-2P, T2 PE-68386NL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

Commit message: - changed the connectors for the temperature sensors
Parts:
- removed P10: T29-32, alexmod:DSUB15HD_90
- removed P5: T9-12, alexmod:DSUB15HD_90
- removed P6: T13-16, alexmod:DSUB15HD_90
- removed P7: T17-20, alexmod:DSUB15HD_90
- removed P8: T21-24, alexmod:DSUB15HD_90
- removed P9: T25-28, alexmod:DSUB15HD_90
- P1, P2: footprint Connectors_Phoenix:PhoenixContact_MC-G_02x3.50mm_Angled -> alexmod:Molex_0678007001
- P3: value T1-4 -> Temp 1-16; footprint alexmod:DSUB15HD_90 -> alexmod:Ampenol_HFW22R
- P4: value T5-8 -> Temp 17-32; footprint alexmod:DSUB15HD_90 -> alexmod:Ampenol_HFW22R
- moved P1 407.6 mm to (455.4, 123.2)
- moved P2 403.3 mm to (54.0, 120.8)
- moved P4 122.2 mm to (318.5, 117.2), turned to 0 degrees
- moved P3 55.9 mm to (188.2, 68.8)
- moved R185 9.34 mm to (262.5, 86.8)
- moved R183 8.37 mm to (273.8, 76.2), turned to 270 degrees
- moved R121 8.11 mm to (436.5, 62.0), turned to 90 degrees
- moved R122 7.11 mm to (434.5, 62.0), turned to 90 degrees
- moved R186 6.00 mm to (262.5, 84.2), turned to 0 degrees
- moved R184 6.00 mm to (262.5, 89.2), turned to 0 degrees
- moved C59 4.55 mm to (425.1, 110.5), turned to 180 degrees
- moved R120 3.85 mm to (441.6, 70.4)
- moved R123 3.85 mm to (444.6, 70.4)
- moved C60 0.76 mm to (443.1, 110.5), turned to 180 degrees
- moved C58 0.50 mm to (431.0, 62.0)
Connections:
- P1 pad 1: /BMS1/BUS_I_P -> /SHIELD
- P2 pad 1: /BMS1/BUS_I_P -> /SHIELD
- P3 pad 1: /BMS1/5V_1 -> /BMS1/BMS1-
- P3 pad 10: (no net) -> /BMS1/T7
- P3 pad 11: /BMS1/BMS1- -> /BMS1/T8
- P3 pad 12: /BMS1/BMS1- -> /BMS1/T9
- P3 pad 13: /BMS1/BMS1- -> /BMS1/T10
- P3 pad 14: /BMS1/BMS1- -> /BMS1/T11
- P3 pad 15: /BMS1/BMS1- -> /BMS1/T12
- P3 pad 2: /BMS1/5V_1 -> /BMS1/BMS1-
- P3 pad 4: /BMS1/5V_1 -> /BMS1/T1
- P3 pad 5: /BMS1/5V_1 -> /BMS1/T2
- P3 pad 6: /BMS1/T1 -> /BMS1/T3
- P3 pad 7: /BMS1/T2 -> /BMS1/T4
- P3 pad 8: /BMS1/T3 -> /BMS1/T5
- P3 pad 9: /BMS1/T4 -> /BMS1/T6
- P4 pad 1: /BMS1/5V_1 -> /BMS1/BMS1+
- P4 pad 10: (no net) -> /BMS2/T10
- P4 pad 11: /BMS1/BMS1- -> /BMS2/T9
- P4 pad 12: /BMS1/BMS1- -> /BMS2/T8
- P4 pad 13: /BMS1/BMS1- -> /BMS2/T7
- P4 pad 14: /BMS1/BMS1- -> /BMS2/T6
- P4 pad 15: /BMS1/BMS1- -> /BMS2/T5
- P4 pad 2: /BMS1/5V_1 -> /BMS1/BMS1+
- P4 pad 3: /BMS1/5V_1 -> /BMS2/5V_2
- P4 pad 4: /BMS1/5V_1 -> /BMS2/T16
- P4 pad 5: /BMS1/5V_1 -> /BMS2/T15
- P4 pad 6: /BMS1/T5 -> /BMS2/T14
- P4 pad 7: /BMS1/T6 -> /BMS2/T13
- P4 pad 8: /BMS1/T7 -> /BMS2/T12
- P4 pad 9: /BMS1/T8 -> /BMS2/T11
Routing:
- net /SHIELD: track 0.00 -> 576.9 mm, vias 0 -> 2
- net Net-(J17-Pad1): track 275.2 -> 48.9 mm, vias 2 -> 3
- net /BMS1/BMS1+: track 682.4 -> 507.5 mm, vias 20 -> 21
- net Net-(J26-Pad1): track 541.8 -> 404.9 mm, vias 1 -> 2
- net Net-(J27-Pad1): track 192.5 -> 61.6 mm
- net /BMS1/5V_1: track 331.1 -> 202.7 mm, vias 7 -> 9
- net /BMS1/T1: track 137.7 -> 51.3 mm, vias 1 -> 0
- net /BMS1/T2: track 132.1 -> 49.7 mm, vias 1 -> 0
- net Net-(J16-Pad1): track 204.2 -> 124.7 mm, vias 2 -> 3
- net /BMS1/T11: track 176.6 -> 97.3 mm, vias 1 -> 2
- net /BMS2/T13: track 82.4 -> 160.7 mm, vias 0 -> 2
- net /BMS1/T9: track 168.3 -> 92.0 mm, vias 1 -> 2
- net /BMS2/5V_2: track 389.2 -> 313.1 mm
- net /BMS1/T3: track 132.5 -> 57.8 mm, vias 1 -> 2
- net /BMS1/T4: track 123.2 -> 49.8 mm, vias 1 -> 0
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Other:
- net class Default: via_drill 0.4 -> 0.3
- rule pad_to_mask_clearance: 0.2 -> 0.08
- board text added: "SCHRÖDER ENGINEERING 20170813 V1.0 NeoBMS E-TEAM"
